Commit message: initial commit

File: src/follow_bot/urdf/follow_bot.urdf.xacro (robot description, xacro)
@@ -136,5 +136,6 @@
   <!-- Colour -->
   <gazebo reference="base_link">
-  <material name="blue" />
+  <!-- <material name="blue" /> -->
+    <material>Gazebo/Blue</material>
   </gazebo>
 </robot>
